File: pcb_design/Power.sch (KiCad schematic (older format))
At the start: 48 parts, among them U2 TC2117, U3 DRV8302

Commit message: Fix inverted diff signals
Signed-off-by: Marcos Chaparro <mchaparro@paltatech.com>
Parts:
- removed C1, C39, C40, C43, C44, C49, C8, C9: 10u,50V, CRF1:SMD-1206, symbol C-RESCUE-BLDC_4
- removed C18, C20, C23, C24, C26, C52: 2.2u, CRF1:SMD-0603_c, symbol C-RESCUE-BLDC_4
- removed C19: 120p, CRF1:SMD-0603_c, symbol C-RESCUE-BLDC_4
- removed C21: 6.8n, CRF1:SMD-0603_c, symbol C-RESCUE-BLDC_4
- removed C22: 22n, CRF1:SMD-0603_c, symbol C-RESCUE-BLDC_4
- removed C25, C33: 100u, w_smd_cap:c_tant_B, symbol CP1-RESCUE-BLDC_4
- removed C27: 100n, CRF1:SMD-0603_c, symbol C-RESCUE-BLDC_4
- removed C28, C29, C30: 220n, CRF1:SMD-0603_c, symbol C-RESCUE-BLDC_4
- removed C34, C36: 2.2n, CRF1:SMD-0603_c, symbol C-RESCUE-BLDC_4
- removed C37: 15u,100V, w_smd_cap:c_2220, symbol C-RESCUE-BLDC_4
- removed C51: 15u, 100v, w_smd_cap:c_2220, symbol C-RESCUE-BLDC_4
- removed D4: DIODESCH, Diodes_SMD:SMA_Handsoldering, symbol DIODESCH
- removed D5: TVS 5V, w_smd_diode:do214ac, symbol DIODE
- removed L1: 22u, w_smd_inductors:inductor_smd_8x5mm, symbol INDUCTOR
- removed R17: 18k, CRF1:SMD-0603_r, symbol R-RESCUE-BLDC_4
- removed R18: 3k3, CRF1:SMD-0603_r, symbol R-RESCUE-BLDC_4
- removed R19: 15k, CRF1:SMD-0603_r, symbol R-RESCUE-BLDC_4
- removed R20: 10k, CRF1:SMD-0603_r, symbol R-RESCUE-BLDC_4
- removed R21: 220k, CRF1:SMD-0603_r, symbol R-RESCUE-BLDC_4
- removed R23, R26, R32: 39k, CRF1:SMD-0603_r, symbol R-RESCUE-BLDC_4
- removed R24, R27, R33: 2k2, CRF1:SMD-0603_r, symbol R-RESCUE-BLDC_4
- removed R25: 1M, CRF1:SMD-0603_r, symbol R-RESCUE-BLDC_4
- removed R48, R49, R50, R51: 100R, CRF1:SMD-0603_r, symbol R-RESCUE-BLDC_4
- removed U2: TC2117, CRF1:SOT-223, symbol NCP1117ST33T3G
- removed U3: DRV8302, CRF1:TSSOP-56-PP, symbol DRV8302
- added C39, C43: 1uF 50v, IPC7351-Nominal:CAPC2012X70, symbol C-0805
- added C40, C42: 180nF, IPC7351-Nominal:CAPC1608X55, symbol C-0603
- added C44: 680pF, IPC7351-Nominal:CAPC2012X70, symbol C-0805
- added C45: 2.2uF 50v, IPC7351-Nominal:CAPC3216X70, symbol C-1206
- added C46, C47, C49, C52: 22uF 10v, IPC7351-Nominal:CAPC3216X70, symbol C-1206
- added C48, C50: 22uF, IPC7351-Nominal:CAPC2012X70, symbol C-0805
- added C5: 10uF 35v, IPC7351-Nominal:CAPC3216X70, symbol C-1206
- added C51: 100nF, IPC7351-Nominal:CAPC1608X55, symbol C-0603
- added C6: 4.7uF 50v tant, IPC7351-Nominal:CAPMP7343X310, symbol C-TANT-7343-31
- added C7: 750pF, IPC7351-Nominal:CAPC2012X70, symbol C-0805
- added D15, D17: SS16, IPC7351-Nominal:DIOM5326X292, symbol SS16
- added D16: 30BQ100TR, IPC7351-Nominal:DIOM7959X265, symbol MBRS360
- added DZ1: 1SMB18CAT, w_smd_diode:do214aa, symbol ESD9L5.0ST5G
- added L1, L3: 22uH 5.2A, manuf:BOURNS-SRR1210, symbol L-1210
- added L2: 27uH, manuf:BOURNS-SDR1307, symbol L-BOURNS-SRN1060
- added Q1: BSC340N08, manuf:TEXAS-Q5A, symbol CSD18503Q5A
- added Q3: AO4805, IPC7351-Nominal:SOIC127P600X175-8, symbol AO4805
- added R12: 1.78k, IPC7351-Nominal:RESC1608X50, symbol R-0603
- added R13: 33.2k, IPC7351-Nominal:RESC1608X50, symbol R-0603
- added R142, R143, R75: 10k, IPC7351-Nominal:RESC1608X50, symbol R-0603
- added R22: 100R, IPC7351-Nominal:RESC1608X50, symbol R-0603
- added R37: 18mOhm, IPC7351-Nominal:CAPC1632X76, symbol R-0612
- added R74: 180k, IPC7351-Nominal:RESC1608X50, symbol R-0603
- added RT1: FUSE 5A SLOW, IPC7351-Most:RESC3216X60, symbol POLYFUSE-30R500
- added RT2: POLYFUSE 1A, IPC7351-Most:RESC3216X60, symbol POLYFUSE-30R500
- added U11: LM3488, IPC7351-Nominal:SOP65P490X109-8, symbol LM3488
- added U13: LM1117IMP-v.v, smd-semi:SOT-223, symbol LM1117IMP-v.v
- added U9: LM22676QTJ-5.0, manuf:TO-263-7-TEXAS, symbol LM22676QTJ-5.0
Connections:
- net labels added: +24, +3.3, +5, 12v_in
- net labels removed: +5V, BR_SO1, BR_SO2, DC_CAL, EN_GATE, FAULT, H1, H1_LOW, H1_VS, H2, H2_LOW, H2_VS, H3, H3_LOW, H3_VS, L1, L2, L3, M_H1, M_H2, M_H3, M_L1, M_L2, M_L3, SENS1, SENS2, SENS3, SH1_A, SH1_B, SH2_A, SH2_B, VCC, V_SUPPLY
- wire segments 189 -> 111
- no-connect marks 4 -> 1
Other:
- note added: "3.3v LDO regulator"
- note added: "9v-30v to 24v 1A SMPS"
- note added: "9v-30v to 5.0v 3A SMPS"
- note added: "Pretty much a textual copy\nof a web bench design"
- note added: "Reverse polarity\nprotection"
- note added: "Should the MCU\nenable this supply?"
- note added: "^ this footprint was horribly wrong"
- note added: "this tantalum cap\nis really bad"
- note removed: "3.3v regulator\nfor the logic"
- note removed: "MCU must sense the\nvoltage at each phase"
